Commit message: while debugging

File: open_manipulator_6dof_description/urdf/open_manipulator_6dof.gazebo.xacro (robot description, xacro)
@@ -26,4 +26,8 @@
   <!-- Link5 -->
   <RefLink ref="link5"/>
+  <!-- Link6 -->
+  <RefLink ref="link6"/>
+  <!-- Link7 -->
+  <RefLink ref="link7"/>
   <!-- gripper_link -->
   <RefLink ref="gripper_link"/>

File: open_manipulator_6dof_description/urdf/open_manipulator_6dof.urdf.xacro (robot description, xacro)
@@ -62,5 +62,5 @@
     <parent link="link1"/>
     <child link="link2"/>
-    <origin xyz="0.0 0.0 0.0" rpy="0 0 0"/>
+    <origin xyz="0.012 0.0 0.017" rpy="0 0 0"/>
     <axis xyz="0 0 1"/>
     <limit velocity="4.8" effort="1" lower="${-pi*0.9}" upper="${pi*0.9}" />
@@ -71,5 +71,5 @@
   <link name="link2">
     <visual>
-      <origin xyz="0 0 0.0" rpy="0 0 0"/>
+      <origin xyz="0 0 0.019" rpy="0 0 0"/>
       <geometry>
         <mesh filename="package://open_manipulator_6dof_description/meshes/chain_link2.stl" scale="0.001 0.001 0.001"/>
@@ -78,5 +78,5 @@
     </visual>
     <collision>
-      <origin xyz="0 0 0.0" rpy="0 0 0"/>
+      <origin xyz="0 0 0.019" rpy="0 0 0"/>
       <geometry>
         <mesh filename="package://open_manipulator_6dof_description/meshes/chain_link2.stl" scale="0.001 0.001 0.001"/>
@@ -102,5 +102,5 @@
     <parent link="link2"/>
     <child link="link3"/>
-    <origin xyz="0.0 0.0 0.0" rpy="0 0 0"/>
+    <origin xyz="0.0 0.0 0.0595" rpy="0 0 0"/>
     <axis xyz="0 1 0"/>
     <limit velocity="4.8" effort="1" lower="${-pi*0.57}" upper="${pi*0.5}" />
@@ -142,5 +142,5 @@
     <parent link="link3"/>
     <child link="link4"/>
-    <origin xyz="0.024 0 0.128" rpy="0 0 0"/>
+    <origin xyz="0.0 0 0.124" rpy="0 0 0"/>
     <axis xyz="0 1 0"/>
     <limit velocity="4.8" effort="1" lower="${-pi*0.3}" upper="${pi*0.44}" />
@@ -182,6 +182,6 @@
     <parent link="link4"/>
     <child link="link5"/>
-    <origin xyz="0.124 0.0 0.0" rpy="0 0 0"/>
-    <axis xyz="0 1 0"/>
+    <origin xyz="0.0 0.0 0.045" rpy="0 0 0"/>
+    <axis xyz="0 0 1"/>
     <limit velocity="4.8" effort="1" lower="${-pi*0.57}" upper="${pi*0.65}" />
   </joint>
@@ -191,5 +191,5 @@
   <link name="link5">
     <visual>
-      <origin xyz="0 0 0" rpy="0 0 0"/>
+      <origin xyz="0 0 0.019" rpy="0 0 0"/>
       <geometry>
         <mesh filename="package://open_manipulator_6dof_description/meshes/chain_link5.stl" scale="0.001 0.001 0.001"/>
@@ -198,7 +198,87 @@
     </visual>
     <collision>
-      <origin xyz="0 0 0" rpy="0 0 0"/>
+      <origin xyz="0 0 0.019" rpy="0 0 0"/>
       <geometry>
         <mesh filename="package://open_manipulator_6dof_description/meshes/chain_link5.stl" scale="0.001 0.001 0.001"/>
+      </geometry>
+    </collision>
+<!--    <inertial>
+      <origin xyz="0 0 0" />
+      <mass value="0.141" />
+      <inertia ixx="0.1" ixy="0.0" ixz="0.0"
+               iyy="0.1" iyz="0.0"
+               izz="0.1" />
+    </inertial>-->
+     <inertial>
+      <origin xyz="4.4206755e-02 3.6839985e-07 8.9142216e-03" />
+      <mass value="1.4327573e-01" />
+      <inertia ixx="8.0870749e-05" ixy="0.0" ixz="-1.0157896e-06"
+               iyy="7.5980465e-05" iyz="0.0"
+               izz="9.3127351e-05" />
+    </inertial>
+  </link>
+  <!--  Joint 5 -->
+  <joint name="joint5" type="revolute">
+    <parent link="link5"/>
+    <child link="link6"/>
+    <origin xyz="0.0 0.0 0.0595" rpy="0 0 0"/>
+    <axis xyz="0 1 0"/>
+    <limit velocity="4.8" effort="1" lower="${-pi*0.57}" upper="${pi*0.65}" />
+  </joint>
+  <!-- Transmission 5 -->
+  <xacro:SimpleTransmission n="5" joint="joint5" />
+  <!--  Link 6 -->
+  <link name="link6">
+    <visual>
+      <origin xyz="0 0 0.0" rpy="0 0 0"/>
+      <geometry>
+        <mesh filename="package://open_manipulator_6dof_description/meshes/chain_link6.stl" scale="0.001 0.001 0.001"/>
+      </geometry>
+      <material name="grey"/>
+    </visual>
+    <collision>
+      <origin xyz="0 0 0.0" rpy="0 0 0"/>
+      <geometry>
+        <mesh filename="package://open_manipulator_6dof_description/meshes/chain_link6.stl" scale="0.001 0.001 0.001"/>
+      </geometry>
+    </collision>
+<!--    <inertial>
+      <origin xyz="0 0 0" />
+      <mass value="0.141" />
+      <inertia ixx="0.1" ixy="0.0" ixz="0.0"
+               iyy="0.1" iyz="0.0"
+               izz="0.1" />
+    </inertial>-->
+     <inertial>
+      <origin xyz="4.4206755e-02 3.6839985e-07 8.9142216e-03" />
+      <mass value="1.4327573e-01" />
+      <inertia ixx="8.0870749e-05" ixy="0.0" ixz="-1.0157896e-06"
+               iyy="7.5980465e-05" iyz="0.0"
+               izz="9.3127351e-05" />
+    </inertial>
+  </link>
+  <!--  Joint 6 -->
+  <joint name="joint6" type="revolute">
+    <parent link="link6"/>
+    <child link="link7"/>
+    <origin xyz="0.0 0.0 0.0305" rpy="0 0 0"/> <!--0.0475 -->
+    <axis xyz="0 0 1"/>
+    <limit velocity="4.8" effort="1" lower="${-pi*0.57}" upper="${pi*0.65}" />
+  </joint>
+  <!-- Transmission 6 -->
+  <xacro:SimpleTransmission n="6" joint="joint6" />
+  <!--  Link 7 -->
+  <link name="link7">
+    <visual>
+      <origin xyz="0 0 0.0" rpy="0 0 0"/>
+      <geometry>
+        <mesh filename="package://open_manipulator_6dof_description/meshes/chain_link7.stl" scale="0.001 0.001 0.001"/>
+      </geometry>
+      <material name="grey"/>
+    </visual>
+    <collision>
+      <origin xyz="0 0 0.0" rpy="0 0 0"/>
+      <geometry>
+        <mesh filename="package://open_manipulator_6dof_description/meshes/chain_link7.stl" scale="0.001 0.001 0.001"/>
       </geometry>
     </collision>
@@ -250,12 +330,12 @@
   <!--  Gripper joint -->
   <joint name="gripper" type="prismatic">
-    <parent link="link5"/>
+    <parent link="link7"/>
     <child link="gripper_link"/>
-    <origin xyz="0.0817 0.019 0.0" rpy="0 0 0"/>
+    <origin xyz="0.0 0.019 0.1" rpy="0 0 0"/>
     <axis xyz="0 1 0"/>
-    <limit velocity="4.8" effort="1" lower="-0.010" upper="0.019" />
-  </joint>
-  <!-- Transmission 5 -->
-  <xacro:SimpleTransmission n="5" joint="gripper" />
+    <limit velocity="4.8" effort="1" lower="-0.010" upper="0.010" />
+  </joint>
+  <!-- Transmission 7 -->
+  <xacro:SimpleTransmission n="7" joint="gripper" />
   <!--  Gripper link sub -->
   <link name="gripper_link_sub">
@@ -290,17 +370,17 @@
   <!--  Gripper joint sub -->
   <joint name="gripper_sub" type="prismatic">
-    <parent link="link5"/>
+    <parent link="link7"/>
     <child link="gripper_link_sub"/>
-    <origin xyz="0.0817 -0.019 0" rpy="0 0 0"/>
+    <origin xyz="0.0 -0.019 0.1" rpy="0 0 0"/>
     <axis xyz="0 -1 0"/>
-    <limit velocity="4.8" effort="1" lower="-0.010" upper="0.019" />
+    <limit velocity="4.8" effort="1" lower="-0.010" upper="0.010" />
     <mimic joint="gripper" multiplier="1"/>
   </joint>
-  <!-- Transmission 6 -->
-  <xacro:SimpleTransmission n="6" joint="gripper_sub" />
+  <!-- Transmission 8 -->
+  <xacro:SimpleTransmission n="8" joint="gripper_sub" />
   <!-- end effector joint -->
   <joint name="end_effector_joint" type="fixed">
-    <origin xyz="0.126 0.0 0.0" rpy="0 0 0"/>
-    <parent link="link5"/>
+    <origin xyz="0.0 0.0 0.115" rpy="0 0 0"/>
+    <parent link="link7"/>
     <child link="end_effector_link"/>
   </joint>
