Commit message: update urdf

File: open_manipulator_6dof_description/urdf/open_manipulator_6dof.urdf.xacro (robot description, xacro)
@@ -1,9 +1,9 @@
 <?xml version="1.0"?>
-<!-- Open_Manipulator Chain -->
-<robot name="open_manipulator" xmlns:xacro="http://ros.org/wiki/xacro">
+<!-- Open_Manipulator 6DOF -->
+<robot name="open_manipulator_6dof" xmlns:xacro="http://ros.org/wiki/xacro">
   <!-- Import all Gazebo-customization elements, including Gazebo colors -->
-  <xacro:include filename="$(find open_manipulator_description)/urdf/open_manipulator.gazebo.xacro" />
+  <xacro:include filename="$(find open_manipulator_6dof_description)/urdf/open_manipulator_6dof.gazebo.xacro" />
   <!-- Import Rviz colors -->
-  <xacro:include filename="$(find open_manipulator_description)/urdf/materials.xacro" />
+  <xacro:include filename="$(find open_manipulator_6dof_description)/urdf/materials.xacro" />
   <!-- Transmission macro -->
   <xacro:macro name="SimpleTransmission" params="joint n">
@@ -33,15 +33,15 @@
       <origin xyz="0 0 0" rpy="0 0 0"/>
       <geometry>
-        <mesh filename="package://open_manipulator_description/meshes/chain_link1.stl" scale="0.001 0.001 0.001"/>
-      </geometry>
-      <material name="grey"/>
-    </visual>
-    <collision>
-      <origin xyz="0 0 0" rpy="0 0 0"/>
-      <geometry>
-        <mesh filename="package://open_manipulator_description/meshes/chain_link1.stl" scale="0.001 0.001 0.001"/>
-      </geometry>
-    </collision>
-    <inertial>
+        <mesh filename="package://open_manipulator_6dof_description/meshes/chain_link1.stl" scale="0.001 0.001 0.001"/>
+      </geometry>
+      <material name="grey"/>
+    </visual>
+    <collision>
+      <origin xyz="0 0 0" rpy="0 0 0"/>
+      <geometry>
+        <mesh filename="package://open_manipulator_6dof_description/meshes/chain_link1.stl" scale="0.001 0.001 0.001"/>
+      </geometry>
+    </collision>
+<!--    <inertial>
       <origin xyz="0 0 0" />
       <mass value="0.082" />
@@ -49,6 +49,6 @@
                iyy="0.1" iyz="0.0"
                izz="0.1" />
-    </inertial>
-    <!-- <inertial>
+    </inertial>-->
+     <inertial>
       <origin xyz="3.0876154e-04 0.0000000e+00 -1.2176461e-04" />
       <mass value="7.9119962e-02" />
@@ -56,5 +56,5 @@
                iyy="2.1898364e-05" iyz="0.0"
                izz="1.9267361e-05" />
-    </inertial> -->
+    </inertial>
   </link>
   <!-- Joint 1 -->
@@ -62,5 +62,5 @@
     <parent link="link1"/>
     <child link="link2"/>
-    <origin xyz="0.012 0.0 0.017" rpy="0 0 0"/>
+    <origin xyz="0.0 0.0 0.0" rpy="0 0 0"/>
     <axis xyz="0 0 1"/>
     <limit velocity="4.8" effort="1" lower="${-pi*0.9}" upper="${pi*0.9}" />
@@ -71,17 +71,17 @@
   <link name="link2">
     <visual>
-      <origin xyz="0 0 0.018" rpy="0 0 0"/>
-      <geometry>
-        <mesh filename="package://open_manipulator_description/meshes/chain_link2.stl" scale="0.001 0.001 0.001"/>
-      </geometry>
-      <material name="grey"/>
-    </visual>
-    <collision>
-      <origin xyz="0 0 0.018" rpy="0 0 0"/>
-      <geometry>
-        <mesh filename="package://open_manipulator_description/meshes/chain_link2.stl" scale="0.001 0.001 0.001"/>
-      </geometry>
-    </collision>
-    <inertial>
+      <origin xyz="0 0 0.0" rpy="0 0 0"/>
+      <geometry>
+        <mesh filename="package://open_manipulator_6dof_description/meshes/chain_link2.stl" scale="0.001 0.001 0.001"/>
+      </geometry>
+      <material name="grey"/>
+    </visual>
+    <collision>
+      <origin xyz="0 0 0.0" rpy="0 0 0"/>
+      <geometry>
+        <mesh filename="package://open_manipulator_6dof_description/meshes/chain_link2.stl" scale="0.001 0.001 0.001"/>
+      </geometry>
+    </collision>
+<!--    <inertial>
       <origin xyz="0 0 0" />
       <mass value="0.098" />
@@ -89,6 +89,6 @@
                iyy="0.1" iyz="0.0"
                izz="0.1" />
-    </inertial>
-    <!-- <inertial>
+    </inertial>-->
+     <inertial>
       <origin xyz="-3.0184870e-04 5.4043684e-04 ${0.018 + 2.9433464e-02}" />
       <mass value="9.8406837e-02" />
@@ -96,5 +96,5 @@
                iyy="3.2689329e-05" iyz="2.8511935e-08"
                izz="1.8850320e-05" />
-    </inertial> -->
+    </inertial>
   </link>
   <!--  Joint 2 -->
@@ -102,5 +102,5 @@
     <parent link="link2"/>
     <child link="link3"/>
-    <origin xyz="0.0 0.0 0.058" rpy="0 0 0"/>
+    <origin xyz="0.0 0.0 0.0" rpy="0 0 0"/>
     <axis xyz="0 1 0"/>
     <limit velocity="4.8" effort="1" lower="${-pi*0.57}" upper="${pi*0.5}" />
@@ -113,15 +113,15 @@
       <origin xyz="0 0 0" rpy="0 0 0"/>
       <geometry>
-        <mesh filename="package://open_manipulator_description/meshes/chain_link3.stl" scale="0.001 0.001 0.001"/>
-      </geometry>
-      <material name="grey"/>
-    </visual>
-    <collision>
-      <origin xyz="0 0 0" rpy="0 0 0"/>
-      <geometry>
-        <mesh filename="package://open_manipulator_description/meshes/chain_link3.stl" scale="0.001 0.001 0.001"/>
-      </geometry>
-    </collision>
-    <inertial>
+        <mesh filename="package://open_manipulator_6dof_description/meshes/chain_link3.stl" scale="0.001 0.001 0.001"/>
+      </geometry>
+      <material name="grey"/>
+    </visual>
+    <collision>
+      <origin xyz="0 0 0" rpy="0 0 0"/>
+      <geometry>
+        <mesh filename="package://open_manipulator_6dof_description/meshes/chain_link3.stl" scale="0.001 0.001 0.001"/>
+      </geometry>
+    </collision>
+<!--    <inertial>
       <origin xyz="0 0 0" />
       <mass value="0.136" />
@@ -129,6 +129,6 @@
                iyy="0.1" iyz="0.0"
                izz="0.1" />
-    </inertial>
-    <!-- <inertial>
+    </inertial>-->
+     <inertial>
       <origin xyz="1.0308393e-02 3.7743363e-04 1.0170197e-01" />
       <mass value="1.3850917e-01" />
@@ -136,5 +136,5 @@
                iyy="3.4290447e-04" iyz="-1.5717516e-06"
                izz="6.0346498e-05" />
-    </inertial> -->
+    </inertial>
   </link>
   <!--  Joint 3 -->
@@ -153,15 +153,15 @@
       <origin xyz="0 0 0" rpy="0 0 0"/>
       <geometry>
-        <mesh filename="package://open_manipulator_description/meshes/chain_link4.stl" scale="0.001 0.001 0.001"/>
-      </geometry>
-      <material name="grey"/>
-    </visual>
-    <collision>
-      <origin xyz="0 0 0" rpy="0 0 0"/>
-      <geometry>
-        <mesh filename="package://open_manipulator_description/meshes/chain_link4.stl" scale="0.001 0.001 0.001"/>
-      </geometry>
-    </collision>
-    <inertial>
+        <mesh filename="package://open_manipulator_6dof_description/meshes/chain_link4.stl" scale="0.001 0.001 0.001"/>
+      </geometry>
+      <material name="grey"/>
+    </visual>
+    <collision>
+      <origin xyz="0 0 0" rpy="0 0 0"/>
+      <geometry>
+        <mesh filename="package://open_manipulator_6dof_description/meshes/chain_link4.stl" scale="0.001 0.001 0.001"/>
+      </geometry>
+    </collision>
+<!--    <inertial>
       <origin xyz="0 0 0" />
       <mass value="0.131" />
@@ -169,6 +169,6 @@
                iyy="0.1" iyz="0.0"
                izz="0.1" />
-    </inertial>
-    <!-- <inertial>
+    </inertial>-->
+     <inertial>
       <origin xyz="9.0909590e-02 3.8929816e-04 2.2413279e-04" />
       <mass value="1.3274562e-01" />
@@ -176,5 +176,5 @@
                iyy="2.4230292e-04" iyz="1.1559550e-08"
                izz="2.5155057e-04" />
-    </inertial> -->
+    </inertial>
   </link>
   <!--  Joint 4 -->
@@ -193,15 +193,15 @@
       <origin xyz="0 0 0" rpy="0 0 0"/>
       <geometry>
-        <mesh filename="package://open_manipulator_description/meshes/chain_link5.stl" scale="0.001 0.001 0.001"/>
-      </geometry>
-      <material name="grey"/>
-    </visual>
-    <collision>
-      <origin xyz="0 0 0" rpy="0 0 0"/>
-      <geometry>
-        <mesh filename="package://open_manipulator_description/meshes/chain_link5.stl" scale="0.001 0.001 0.001"/>
-      </geometry>
-    </collision>
-    <inertial>
+        <mesh filename="package://open_manipulator_6dof_description/meshes/chain_link5.stl" scale="0.001 0.001 0.001"/>
+      </geometry>
+      <material name="grey"/>
+    </visual>
+    <collision>
+      <origin xyz="0 0 0" rpy="0 0 0"/>
+      <geometry>
+        <mesh filename="package://open_manipulator_6dof_description/meshes/chain_link5.stl" scale="0.001 0.001 0.001"/>
+      </geometry>
+    </collision>
+<!--    <inertial>
       <origin xyz="0 0 0" />
       <mass value="0.141" />
@@ -209,6 +209,6 @@
                iyy="0.1" iyz="0.0"
                izz="0.1" />
-    </inertial>
-    <!-- <inertial>
+    </inertial>-->
+     <inertial>
       <origin xyz="4.4206755e-02 3.6839985e-07 8.9142216e-03" />
       <mass value="1.4327573e-01" />
@@ -216,5 +216,5 @@
                iyy="7.5980465e-05" iyz="0.0"
                izz="9.3127351e-05" />
-    </inertial> -->
+    </inertial>
   </link>
   <!--  Gripper link -->
@@ -223,5 +223,5 @@
       <origin xyz="0.0 0.0 0" rpy="0 0 0"/>
       <geometry>
-        <mesh filename="package://open_manipulator_description/meshes/chain_link_grip_l.stl" scale="0.001 0.001 0.001"/>
+        <mesh filename="package://open_manipulator_6dof_description/meshes/chain_link_grip_l.stl" scale="0.001 0.001 0.001"/>
       </geometry>
       <material name="grey"/>
@@ -230,5 +230,5 @@
       <origin xyz="0.0 0.0 0" rpy="0 0 0"/>
       <geometry>
-        <mesh filename="package://open_manipulator_description/meshes/chain_link_grip_l.stl" scale="0.001 0.001 0.001"/>
+        <mesh filename="package://open_manipulator_6dof_description/meshes/chain_link_grip_l.stl" scale="0.001 0.001 0.001"/>
       </geometry>
     </collision>
@@ -236,9 +236,9 @@
       <origin xyz="0 0 0" />
       <mass value="0.017" />
-      <inertia ixx="0.1" ixy="0.0" ixz="0.0"
-               iyy="0.1" iyz="0.0"
-               izz="0.1" />
-    </inertial>
-    <!-- <inertial>
+      <inertia ixx="1.0e-03" ixy="0.0" ixz="0.0"
+               iyy="1.0e-03" iyz="0.0"
+               izz="1.0e-03" />
+    </inertial>
+<!--     <inertial>
       <origin xyz="${0.028 + 8.3720668e-03} ${0.0246 + 9.9696160e-03} -4.2836895e-07" />
       <mass value="3.2218127e-02" />
@@ -246,5 +246,5 @@
                iyy="2.2552871e-05" iyz="-3.1463634e-10"
                izz="1.7605306e-05" />
-    </inertial> -->
+    </inertial>-->
   </link>
   <!--  Gripper joint -->
@@ -263,5 +263,5 @@
       <origin xyz="0.0 -0.0 0" rpy="0 0 0"/>
       <geometry>
-        <mesh filename="package://open_manipulator_description/meshes/chain_link_grip_r.stl" scale="0.001 0.001 0.001"/>
+        <mesh filename="package://open_manipulator_6dof_description/meshes/chain_link_grip_r.stl" scale="0.001 0.001 0.001"/>
       </geometry>
       <material name="grey"/>
@@ -270,5 +270,5 @@
       <origin xyz="0.0 -0.0 0" rpy="0 0 0"/>
       <geometry>
-        <mesh filename="package://open_manipulator_description/meshes/chain_link_grip_r.stl" scale="0.001 0.001 0.001"/>
+        <mesh filename="package://open_manipulator_6dof_description/meshes/chain_link_grip_r.stl" scale="0.001 0.001 0.001"/>
       </geometry>
     </collision>
@@ -276,9 +276,9 @@
       <origin xyz="0 0 0" />
       <mass value="0.017" />
-      <inertia ixx="0.1" ixy="0.0" ixz="0.0"
-               iyy="0.1" iyz="0.0"
-               izz="0.1" />
-    </inertial>
-    <!-- <inertial>
+      <inertia ixx="1.0e-03" ixy="0.0" ixz="0.0"
+               iyy="1.0e-03" iyz="0.0"
+               izz="1.0e-03" />
+    </inertial>
+<!--     <inertial>
       <origin xyz="${0.028 + 8.3720668e-03} ${-0.0246 - 9.9696160e-03} -4.2836895e-07" />
       <mass value="3.2218127e-02" />
@@ -286,5 +286,5 @@
                iyy="2.2552871e-05" iyz="-3.1463634e-10"
                izz="1.7605306e-05" />
-    </inertial> -->
+    </inertial>-->
   </link>
   <!--  Gripper joint sub -->
@@ -301,5 +301,5 @@
   <!-- end effector joint -->
   <joint name="end_effector_joint" type="fixed">
-    <origin xyz="0.130 0.0 0.0" rpy="0 0 0"/>
+    <origin xyz="0.126 0.0 0.0" rpy="0 0 0"/>
     <parent link="link5"/>
     <child link="end_effector_link"/>
@@ -317,5 +317,5 @@
       <origin xyz="0.0 0.0 0.0" rpy="0 0 0"/>
       <mass value="0.001"/>
-      <inertia ixx="1.0" ixy="0.0" ixz="0.0" iyy="1.0" iyz="0.0" izz="1.0" />
+      <inertia ixx="1.0e-06" ixy="0.0" ixz="0.0" iyy="1.0e-06" iyz="0.0" izz="1.0e-06" />
     </inertial>
   </link>

Commit message: update

File: open_manipulator_6dof_description/urdf/open_manipulator_6dof.urdf.xacro (robot description, xacro)
@@ -123,12 +123,12 @@
       </geometry>
     </collision>
+    <inertial>
+      <origin xyz="0 0 0" />
+      <mass value="0.131" />
+      <inertia ixx="0.1" ixy="0.0" ixz="0.0"
+               iyy="0.1" iyz="0.0"
+               izz="0.1" />
+    </inertial>
 <!--    <inertial>
-      <origin xyz="0 0 0" />
-      <mass value="0.136" />
-      <inertia ixx="0.1" ixy="0.0" ixz="0.0"
-               iyy="0.1" iyz="0.0"
-               izz="0.1" />
-    </inertial>-->
-     <inertial>
       <origin xyz="1.0308393e-02 3.7743363e-04 1.0170197e-01" />
       <mass value="1.3850917e-01" />
@@ -136,5 +136,5 @@
                iyy="3.4290447e-04" iyz="-1.5717516e-06"
                izz="6.0346498e-05" />
-    </inertial>
+    </inertial>-->
   </link>
   <!--  Joint 3 -->
@@ -163,12 +163,12 @@
       </geometry>
     </collision>
-<!--    <inertial>
-      <origin xyz="0 0 0" />
-      <mass value="0.131" />
-      <inertia ixx="0.1" ixy="0.0" ixz="0.0"
-               iyy="0.1" iyz="0.0"
-               izz="0.1" />
-    </inertial>-->
-     <inertial>
+    <inertial>
+      <origin xyz="0 0 0" />
+      <mass value="0.098" />
+      <inertia ixx="0.1" ixy="0.0" ixz="0.0"
+               iyy="0.1" iyz="0.0"
+               izz="0.1" />
+    </inertial>
+<!--     <inertial>
       <origin xyz="9.0909590e-02 3.8929816e-04 2.2413279e-04" />
       <mass value="1.3274562e-01" />
@@ -176,5 +176,5 @@
                iyy="2.4230292e-04" iyz="1.1559550e-08"
                izz="2.5155057e-04" />
-    </inertial>
+    </inertial>-->
   </link>
   <!--  Joint 4 -->
@@ -203,12 +203,12 @@
       </geometry>
     </collision>
-<!--    <inertial>
-      <origin xyz="0 0 0" />
-      <mass value="0.141" />
-      <inertia ixx="0.1" ixy="0.0" ixz="0.0"
-               iyy="0.1" iyz="0.0"
-               izz="0.1" />
-    </inertial>-->
-     <inertial>
+    <inertial>
+      <origin xyz="0 0 0" />
+      <mass value="0.098" />
+      <inertia ixx="0.1" ixy="0.0" ixz="0.0"
+               iyy="0.1" iyz="0.0"
+               izz="0.1" />
+    </inertial>
+<!--     <inertial>
       <origin xyz="4.4206755e-02 3.6839985e-07 8.9142216e-03" />
       <mass value="1.4327573e-01" />
@@ -216,5 +216,5 @@
                iyy="7.5980465e-05" iyz="0.0"
                izz="9.3127351e-05" />
-    </inertial>
+    </inertial>-->
   </link>
   <!--  Joint 5 -->
@@ -243,11 +243,11 @@
       </geometry>
     </collision>
-<!--    <inertial>
-      <origin xyz="0 0 0" />
-      <mass value="0.141" />
-      <inertia ixx="0.1" ixy="0.0" ixz="0.0"
-               iyy="0.1" iyz="0.0"
-               izz="0.1" />
-    </inertial>-->
+    <inertial>
+      <origin xyz="0 0 0" />
+      <mass value="0.033" />
+      <inertia ixx="0.1" ixy="0.0" ixz="0.0"
+               iyy="0.1" iyz="0.0"
+               izz="0.1" />
+    </inertial>
      <inertial>
       <origin xyz="4.4206755e-02 3.6839985e-07 8.9142216e-03" />
@@ -262,5 +262,5 @@
     <parent link="link6"/>
     <child link="link7"/>
-    <origin xyz="0.0 0.0 0.0305" rpy="0 0 0"/> <!--0.0475 -->
+    <origin xyz="0.0 0.0 0.0475" rpy="0 0 0"/>
     <axis xyz="0 0 1"/>
     <limit velocity="4.8" effort="1" lower="${-pi*0.57}" upper="${pi*0.65}" />
@@ -283,7 +283,7 @@
       </geometry>
     </collision>
-<!--    <inertial>
-      <origin xyz="0 0 0" />
-      <mass value="0.141" />
+    <inertial>
+      <origin xyz="0 0 0" />
+      <mass value="0.228" />
       <inertia ixx="0.1" ixy="0.0" ixz="0.0"
                iyy="0.1" iyz="0.0"
@@ -332,5 +332,5 @@
     <parent link="link7"/>
     <child link="gripper_link"/>
-    <origin xyz="0.0 0.019 0.1" rpy="0 0 0"/>
+    <origin xyz="0.0 0.019 0.0851" rpy="0 0 0"/>
     <axis xyz="0 1 0"/>
     <limit velocity="4.8" effort="1" lower="-0.010" upper="0.010" />
@@ -372,5 +372,5 @@
     <parent link="link7"/>
     <child link="gripper_link_sub"/>
-    <origin xyz="0.0 -0.019 0.1" rpy="0 0 0"/>
+    <origin xyz="0.0 -0.019 0.0851" rpy="0 0 0"/>
     <axis xyz="0 -1 0"/>
     <limit velocity="4.8" effort="1" lower="-0.010" upper="0.010" />
@@ -381,5 +381,5 @@
   <!-- end effector joint -->
   <joint name="end_effector_joint" type="fixed">
-    <origin xyz="0.0 0.0 0.115" rpy="0 0 0"/>
+    <origin xyz="0.0 0.0 0.130" rpy="0 0 0"/>
     <parent link="link7"/>
     <child link="end_effector_link"/>

Commit message: update urdf

File: open_manipulator_6dof_description/urdf/open_manipulator_6dof.urdf.xacro (robot description, xacro)
@@ -19,4 +19,5 @@
     </transmission>
   </xacro:macro>
+cm
   <!-- World -->
   <link name="world">
@@ -332,5 +333,5 @@
     <parent link="link7"/>
     <child link="gripper_link"/>
-    <origin xyz="0.0 0.019 0.0851" rpy="0 0 0"/>
+    <origin xyz="0.0 0.019 0.0707" rpy="0 0 0"/>
     <axis xyz="0 1 0"/>
     <limit velocity="4.8" effort="1" lower="-0.010" upper="0.010" />
@@ -372,5 +373,5 @@
     <parent link="link7"/>
     <child link="gripper_link_sub"/>
-    <origin xyz="0.0 -0.019 0.0851" rpy="0 0 0"/>
+    <origin xyz="0.0 -0.019 0.0707" rpy="0 0 0"/>
     <axis xyz="0 -1 0"/>
     <limit velocity="4.8" effort="1" lower="-0.010" upper="0.010" />
@@ -381,5 +382,5 @@
   <!-- end effector joint -->
   <joint name="end_effector_joint" type="fixed">
-    <origin xyz="0.0 0.0 0.130" rpy="0 0 0"/>
+    <origin xyz="0.0 0.0 0.115" rpy="0 0 0"/>
     <parent link="link7"/>
     <child link="end_effector_link"/>

Commit message: update

File: open_manipulator_6dof_description/urdf/open_manipulator_6dof.urdf.xacro (robot description, xacro)
@@ -104,5 +104,5 @@
     <origin xyz="0.0 0.0 0.0595" rpy="0 0 0"/>
     <axis xyz="0 1 0"/>
-    <limit velocity="4.8" effort="1" lower="${-pi*0.57}" upper="${pi*0.5}" />
+    <limit velocity="4.8" effort="1" lower="${-pi*0.65}" upper="${pi*0.67}" />
   </joint>
   <!-- Transmission 2 -->
@@ -144,5 +144,5 @@
     <origin xyz="0.0 0 0.124" rpy="0 0 0"/>
     <axis xyz="0 1 0"/>
-    <limit velocity="4.8" effort="1" lower="${-pi*0.3}" upper="${pi*0.44}" />
+    <limit velocity="4.8" effort="1" lower="${-pi*0.60}" upper="${pi*0.68}" />
   </joint>
   <!-- Transmission 3 -->
@@ -184,5 +184,5 @@
     <origin xyz="0.0 0.0 0.045" rpy="0 0 0"/>
     <axis xyz="0 0 1"/>
-    <limit velocity="4.8" effort="1" lower="${-pi*0.57}" upper="${pi*0.65}" />
+    <limit velocity="4.8" effort="1" lower="${-pi*0.9}" upper="${pi*0.9}" />
   </joint>
   <!-- Transmission 4 -->
@@ -224,5 +224,5 @@
     <origin xyz="0.0 0.0 0.0595" rpy="0 0 0"/>
     <axis xyz="0 1 0"/>
-    <limit velocity="4.8" effort="1" lower="${-pi*0.57}" upper="${pi*0.65}" />
+    <limit velocity="4.8" effort="1" lower="${-pi*0.63}" upper="${pi*0.66}" />
   </joint>
   <!-- Transmission 5 -->
@@ -264,5 +264,5 @@
     <origin xyz="0.0 0.0 0.0475" rpy="0 0 0"/>
     <axis xyz="0 0 1"/>
-    <limit velocity="4.8" effort="1" lower="${-pi*0.57}" upper="${pi*0.65}" />
+    <limit velocity="4.8" effort="1" lower="${-pi*0.9}" upper="${pi*0.9}" />
   </joint>
   <!-- Transmission 6 -->
@@ -334,5 +334,5 @@
     <origin xyz="0.0 0.019 0.0707" rpy="0 0 0"/>
     <axis xyz="0 1 0"/>
-    <limit velocity="4.8" effort="1" lower="-0.010" upper="0.010" />
+    <limit velocity="4.8" effort="1" lower="-0.010" upper="0.015" />
   </joint>
   <!-- Transmission 7 -->
@@ -374,5 +374,5 @@
     <origin xyz="0.0 -0.019 0.0707" rpy="0 0 0"/>
     <axis xyz="0 -1 0"/>
-    <limit velocity="4.8" effort="1" lower="-0.010" upper="0.010" />
+    <limit velocity="4.8" effort="1" lower="-0.010" upper="0.015" />
     <mimic joint="gripper" multiplier="1"/>
   </joint>

Commit message: change kinematics variables

File: open_manipulator_6dof_description/urdf/open_manipulator_6dof.urdf.xacro (robot description, xacro)
@@ -224,5 +224,5 @@
     <origin xyz="0.0 0.0 0.0595" rpy="0 0 0"/>
     <axis xyz="0 1 0"/>
-    <limit velocity="4.8" effort="1" lower="${-pi*0.63}" upper="${pi*0.66}" />
+    <limit velocity="4.8" effort="1" lower="${-pi*0.63}" upper="${pi*0.67}" />
   </joint>
   <!-- Transmission 5 -->

Commit message: minor change

File: open_manipulator_6dof_description/urdf/open_manipulator_6dof.urdf.xacro (robot description, xacro)
@@ -332,5 +332,5 @@
     <parent link="link7"/>
     <child link="gripper_link"/>
-    <origin xyz="0.0 0.019 0.0707" rpy="0 0 0"/>
+    <origin xyz="0.0 0.021 0.0707" rpy="0 0 0"/>
     <axis xyz="0 1 0"/>
     <limit velocity="4.8" effort="1" lower="-0.010" upper="0.015" />
@@ -372,5 +372,5 @@
     <parent link="link7"/>
     <child link="gripper_link_sub"/>
-    <origin xyz="0.0 -0.019 0.0707" rpy="0 0 0"/>
+    <origin xyz="0.0 -0.021 0.0707" rpy="0 0 0"/>
     <axis xyz="0 -1 0"/>
     <limit velocity="4.8" effort="1" lower="-0.010" upper="0.015" />

Commit message: update

File: open_manipulator_6dof_description/urdf/open_manipulator_6dof.urdf.xacro (robot description, xacro)
@@ -334,5 +334,5 @@
     <origin xyz="0.0 0.021 0.0707" rpy="0 0 0"/>
     <axis xyz="0 1 0"/>
-    <limit velocity="4.8" effort="1" lower="-0.010" upper="0.015" />
+    <limit velocity="4.8" effort="1" lower="-0.010" upper="0.019" />
   </joint>
   <!-- Transmission 7 -->
@@ -374,5 +374,5 @@
     <origin xyz="0.0 -0.021 0.0707" rpy="0 0 0"/>
     <axis xyz="0 -1 0"/>
-    <limit velocity="4.8" effort="1" lower="-0.010" upper="0.015" />
+    <limit velocity="4.8" effort="1" lower="-0.010" upper="0.019" />
     <mimic joint="gripper" multiplier="1"/>
   </joint>
