Commit message: Support 6axis Jazzy

File: open_manipulator_x_description/ros2_control/open_manipulator_x_system.ros2_control.xacro (robot description, xacro)
@@ -18,23 +18,26 @@
             <plugin>dynamixel_hardware_interface/DynamixelHardware</plugin>
             <param name="port_name">${port_name}</param>
-            <param name="baud_rate">1000000</param>
+            <param name="baud_rate">4000000</param>
             <param name="error_timeout_sec">0.2</param>
             <param name="dynamixel_model_folder">/param/dxl_model</param>
-            <param name="number_of_joints">6</param>
-            <param name="number_of_transmissions">5</param>
+            <param name="number_of_joints">7</param>
+            <param name="number_of_transmissions">7</param>
             <param name="transmission_to_joint_matrix">
-              1, 0, 0, 0, 0,
-              0, 1, 0, 0, 0,
-              0, 0, 1, 0, 0,
-              0, 0, 0, 1, 0,
-              0, 0, 0, 0, 1,
-              0, 0, 0, 0, 0
+              1, 0, 0, 0, 0, 0, 0,
+              0, 1, 0, 0, 0, 0, 0,
+              0, 0, 1, 0, 0, 0, 0,
+              0, 0, 0, 1, 0, 0, 0,
+              0, 0, 0, 0, 1, 0, 0,
+              0, 0, 0, 0, 0, 1, 0,
+              0, 0, 0, 0, 0, 0, 1
             </param>
             <param name="joint_to_transmission_matrix">
-              1, 0, 0, 0, 0, 0,
-              0, 1, 0, 0, 0, 0,
-              0, 0, 1, 0, 0, 0,
-              0, 0, 0, 1, 0, 0,
-              0, 0, 0, 0, 1, 0
+              1, 0, 0, 0, 0, 0, 0,
+              0, 1, 0, 0, 0, 0, 0,
+              0, 0, 1, 0, 0, 0, 0,
+              0, 0, 0, 1, 0, 0, 0,
+              0, 0, 0, 0, 1, 0, 0,
+              0, 0, 0, 0, 0, 1, 0,
+              0, 0, 0, 0, 0, 0, 1
             </param>
             <param name="ros_update_freq">200</param>
@@ -47,5 +50,5 @@
             that operates through a revolute mechanism. If the joint does not require this configuration, this parameter can be removed. -->
             <param name="use_revolute_to_prismatic_gripper">1</param>
-            <param name="revolute_to_prismatic_dxl">dxl5</param>
+            <param name="revolute_to_prismatic_dxl">dxl7</param>
             <param name="revolute_max">-1.52</param>
             <param name="revolute_min">0.92</param>
@@ -80,4 +83,16 @@
         <state_interface name="effort"/>
       </joint>
+      <joint name="${prefix}joint5">
+        <command_interface name="position"/>
+        <state_interface name="position"/>
+        <state_interface name="velocity"/>
+        <state_interface name="effort"/>
+      </joint>
+      <joint name="${prefix}joint6">
+        <command_interface name="position"/>
+        <state_interface name="position"/>
+        <state_interface name="velocity"/>
+        <state_interface name="effort"/>
+      </joint>
       <joint name="${prefix}gripper_left_joint">
         <command_interface name="position"/>
@@ -86,12 +101,4 @@
         <state_interface name="effort"/>
       </joint>
-      <joint name="${prefix}gripper_right_joint">
-        <param name="mimic">${prefix}gripper_left_joint</param>
-        <param name="multiplier">1</param>
-        <command_interface name="position"/>
-        <state_interface name="position"/>
-        <state_interface name="velocity"/>
-        <state_interface name="effort"/>
-      </joint>
       <gpio name="dxl1">
         <param name="type">dxl</param>
@@ -109,4 +116,5 @@
         <param name="Profile Acceleration">50</param>
         <param name="Drive Mode">0</param>
+        <param name="Return Delay Time">0</param>
       </gpio>
       <gpio name="dxl2">
@@ -125,4 +133,5 @@
         <param name="Profile Acceleration">50</param>
         <param name="Drive Mode">0</param>
+        <param name="Return Delay Time">0</param>
       </gpio>
       <gpio name="dxl3">
@@ -141,4 +150,5 @@
         <param name="Profile Acceleration">50</param>
         <param name="Drive Mode">0</param>
+        <param name="Return Delay Time">0</param>
       </gpio>
       <gpio name="dxl4">
@@ -157,4 +167,5 @@
         <param name="Profile Acceleration">50</param>
         <param name="Drive Mode">0</param>
+        <param name="Return Delay Time">0</param>
       </gpio>
       <gpio name="dxl5">
@@ -167,4 +178,39 @@
         <state_interface name="Torque Enable"/>
         <state_interface name="Present Input Voltage"/>
+        <param name="Position P Gain">800</param>
+        <param name="Position I Gain">100</param>
+        <param name="Position D Gain">100</param>
+        <param name="Profile Velocity">200</param>
+        <param name="Profile Acceleration">50</param>
+        <param name="Drive Mode">0</param>
+        <param name="Return Delay Time">0</param>
+      </gpio>
+        <gpio name="dxl6">
+        <param name="type">dxl</param>
+        <param name="ID">16</param>
+        <command_interface name="Goal Position"/>
+        <state_interface name="Present Position"/>
+        <state_interface name="Present Velocity"/>
+        <state_interface name="Present Current"/>
+        <state_interface name="Torque Enable"/>
+        <state_interface name="Present Input Voltage"/>
+        <param name="Position P Gain">800</param>
+        <param name="Position I Gain">100</param>
+        <param name="Position D Gain">100</param>
+        <param name="Profile Velocity">200</param>
+        <param name="Profile Acceleration">50</param>
+        <param name="Drive Mode">0</param>
+        <param name="Return Delay Time">0</param>
+      </gpio>
+      <gpio name="dxl7">
+        <param name="type">dxl</param>
+        <param name="ID">17</param>
+        <command_interface name="Goal Position"/>
+        <state_interface name="Present Position"/>
+        <state_interface name="Present Velocity"/>
+        <state_interface name="Present Current"/>
+        <state_interface name="Torque Enable"/>
+        <state_interface name="Present Input Voltage"/>
+        <param name="Return Delay Time">0</param>
       </gpio>
     </ros2_control>

File: open_manipulator_x_description/urdf/open_manipulator_x.urdf.xacro (robot description, xacro)
@@ -19,10 +19,10 @@
         </geometry>
       </collision>
-       <inertial>
+      <inertial>
         <origin xyz="3.0876154e-04 0.0000000e+00 -1.2176461e-04" />
         <mass value="7.9119962e-02" />
         <inertia ixx="1.2505234e-05" ixy="0.0" ixz="-1.7855208e-07"
-                 iyy="2.1898364e-05" iyz="0.0"
-                 izz="1.9267361e-05" />
+                iyy="2.1898364e-05" iyz="0.0"
+                izz="1.9267361e-05" />
       </inertial>
     </link>
@@ -49,10 +49,10 @@
         </geometry>
       </collision>
-       <inertial>
+      <inertial>
         <origin xyz="-3.0184870e-04 5.4043684e-04 ${0.018 + 2.9433464e-02}" />
         <mass value="9.8406837e-02" />
         <inertia ixx="3.4543422e-05" ixy="-1.6031095e-08" ixz="-3.8375155e-07"
-                 iyy="3.2689329e-05" iyz="2.8511935e-08"
-                 izz="1.8850320e-05" />
+                iyy="3.2689329e-05" iyz="2.8511935e-08"
+                izz="1.8850320e-05" />
       </inertial>
     </link>
@@ -62,5 +62,5 @@
       <origin xyz="0.0 0.0 0.0595" rpy="0 0 0"/>
       <axis xyz="0 1 0"/>
-      <limit velocity="4.8" effort="1" lower="${-1.5}" upper="${1.5}" />
+      <limit velocity="4.8" effort="1" lower="${-pi*0.65}" upper="${pi*0.67}" />
       <dynamics damping="0.1"/>
     </joint>
@@ -79,10 +79,10 @@
         </geometry>
       </collision>
-       <inertial>
-        <origin xyz="1.0308393e-02 3.7743363e-04 1.0170197e-01" />
-        <mass value="1.3850917e-01" />
-        <inertia ixx="3.3055381e-04" ixy="-9.7940978e-08" ixz="-3.8505711e-05"
-                 iyy="3.4290447e-04" iyz="-1.5717516e-06"
-                 izz="6.0346498e-05" />
+      <inertial>
+        <origin xyz="0 0 0" />
+        <mass value="0.131" />
+        <inertia ixx="0.1" ixy="0.0" ixz="0.0"
+                iyy="0.1" iyz="0.0"
+                izz="0.1" />
       </inertial>
     </link>
@@ -90,7 +90,7 @@
       <parent link="${prefix}link3"/>
       <child link="${prefix}link4"/>
-      <origin xyz="0.024 0 0.128" rpy="0 0 0"/>
-      <axis xyz="0 1 0"/>
-      <limit velocity="4.8" effort="1" lower="${-1.5}" upper="${1.4}" />
+      <origin xyz="0.0 0 0.124" rpy="0 0 0"/>
+      <axis xyz="0 1 0"/>
+      <limit velocity="4.8" effort="1" lower="${-pi*0.60}" upper="${pi*0.68}" />
       <dynamics damping="0.1"/>
     </joint>
@@ -109,10 +109,10 @@
         </geometry>
       </collision>
-       <inertial>
-        <origin xyz="9.0909590e-02 3.8929816e-04 2.2413279e-04" />
-        <mass value="1.3274562e-01" />
-        <inertia ixx="3.0654178e-05" ixy="-1.2764155e-06" ixz="-2.6874417e-07"
-                 iyy="2.4230292e-04" iyz="1.1559550e-08"
-                 izz="2.5155057e-04" />
+      <inertial>
+        <origin xyz="0 0 0" />
+        <mass value="0.098" />
+        <inertia ixx="0.1" ixy="0.0" ixz="0.0"
+                iyy="0.1" iyz="0.0"
+                izz="0.1" />
       </inertial>
     </link>
@@ -120,12 +120,12 @@
       <parent link="${prefix}link4"/>
       <child link="${prefix}link5"/>
-      <origin xyz="0.124 0.0 0.0" rpy="0 0 0"/>
-      <axis xyz="0 1 0"/>
-      <limit velocity="4.8" effort="1" lower="${-1.7}" upper="${1.97}" />
+      <origin xyz="0.0 0.0 0.045" rpy="0 0 0"/>
+      <axis xyz="0 0 1"/>
+      <limit velocity="4.8" effort="1" lower="${-pi}" upper="${pi}" />
       <dynamics damping="0.1"/>
     </joint>
     <link name="${prefix}link5">
       <visual>
-        <origin xyz="0 0 0" rpy="0 0 0"/>
+        <origin xyz="0 0 0.019" rpy="0 0 0"/>
         <geometry>
           <mesh filename="${meshes_file_direction}/link5.stl" scale="0.001 0.001 0.001"/>
@@ -134,21 +134,79 @@
       </visual>
       <collision>
-        <origin xyz="0 0 0" rpy="0 0 0"/>
+        <origin xyz="0 0 0.019" rpy="0 0 0"/>
         <geometry>
           <mesh filename="${meshes_file_direction}/link5.stl" scale="0.001 0.001 0.001"/>
         </geometry>
       </collision>
-       <inertial>
+      <inertial>
+        <origin xyz="0 0 0" />
+        <mass value="0.098" />
+        <inertia ixx="0.1" ixy="0.0" ixz="0.0"
+                iyy="0.1" iyz="0.0"
+                izz="0.1" />
+      </inertial>
+    </link>
+    <joint name="${prefix}joint5" type="revolute">
+      <parent link="${prefix}link5"/>
+      <child link="${prefix}link6"/>
+      <origin xyz="0.0 0.0 0.0595" rpy="0 0 0"/>
+      <axis xyz="0 1 0"/>
+      <limit velocity="4.8" effort="1" lower="${-pi*0.63}" upper="${pi*0.67}" />
+    </joint>
+    <link name="${prefix}link6">
+      <visual>
+        <origin xyz="0 0 0.0" rpy="0 0 0"/>
+        <geometry>
+          <mesh filename="${meshes_file_direction}/link6.stl" scale="0.001 0.001 0.001"/>
+        </geometry>
+        <material name="grey"/>
+      </visual>
+      <collision>
+        <origin xyz="0 0 0.0" rpy="0 0 0"/>
+        <geometry>
+          <mesh filename="${meshes_file_direction}/link6.stl" scale="0.001 0.001 0.001"/>
+        </geometry>
+      </collision>
+      <inertial>
         <origin xyz="4.4206755e-02 3.6839985e-07 8.9142216e-03" />
         <mass value="1.4327573e-01" />
         <inertia ixx="8.0870749e-05" ixy="0.0" ixz="-1.0157896e-06"
-                 iyy="7.5980465e-05" iyz="0.0"
-                 izz="9.3127351e-05" />
+                iyy="7.5980465e-05" iyz="0.0"
+                izz="9.3127351e-05" />
+      </inertial>
+    </link>
+    <joint name="${prefix}joint6" type="revolute">
+      <parent link="${prefix}link6"/>
+      <child link="${prefix}link7"/>
+      <origin xyz="0.0 0.0 0.0475" rpy="0 0 0"/>
+      <axis xyz="0 0 1"/>
+      <limit velocity="4.8" effort="1" lower="${-pi*0.9}" upper="${pi*0.9}" />
+    </joint>
+    <link name="${prefix}link7">
+      <visual>
+        <origin xyz="0 0 0.0" rpy="0 0 0"/>
+        <geometry>
+          <mesh filename="${meshes_file_direction}/link7.stl" scale="0.001 0.001 0.001"/>
+        </geometry>
+        <material name="grey"/>
+      </visual>
+      <collision>
+        <origin xyz="0 0 0.0" rpy="0 0 0"/>
+        <geometry>
+          <mesh filename="${meshes_file_direction}/link7.stl" scale="0.001 0.001 0.001"/>
+        </geometry>
+      </collision>
+      <inertial>
+        <origin xyz="4.4206755e-02 3.6839985e-07 8.9142216e-03" />
+        <mass value="1.4327573e-01" />
+        <inertia ixx="8.0870749e-05" ixy="0.0" ixz="-1.0157896e-06"
+                iyy="7.5980465e-05" iyz="0.0"
+                izz="9.3127351e-05" />
       </inertial>
     </link>
     <joint name="${prefix}gripper_left_joint" type="prismatic">
-      <parent link="${prefix}link5"/>
+      <parent link="${prefix}link7"/>
       <child link="${prefix}gripper_left_link"/>
-      <origin xyz="0.0817 0.021 0.0" rpy="0 0 0"/>
+      <origin xyz="0.0 0.021 0.0707" rpy="0 0 0"/>
       <axis xyz="0 1 0"/>
       <limit velocity="4.8" effort="1" lower="-0.010" upper="0.019" />
@@ -173,6 +231,6 @@
         <mass value="1.0e-03" />
         <inertia ixx="1.0e-06" ixy="0.0" ixz="0.0"
-                 iyy="1.0e-06" iyz="0.0"
-                 izz="1.0e-06" />
+                iyy="1.0e-06" iyz="0.0"
+                izz="1.0e-06" />
       </inertial>
     </link>
@@ -183,7 +241,7 @@
     <link name="dummy_mimic_fix"/>
     <joint name="${prefix}gripper_right_joint" type="prismatic">
-      <parent link="${prefix}link5"/>
+      <parent link="${prefix}link7"/>
       <child link="${prefix}gripper_right_link"/>
-      <origin xyz="0.0817 -0.021 0" rpy="0 0 0"/>
+      <origin xyz="0.0 -0.021 0.0707" rpy="0 0 0"/>
       <axis xyz="0 -1 0"/>
       <limit velocity="4.8" effort="1" lower="-0.010" upper="0.019" />
@@ -209,12 +267,12 @@
         <mass value="1.0e-03" />
         <inertia ixx="1.0e-06" ixy="0.0" ixz="0.0"
-                 iyy="1.0e-06" iyz="0.0"
-                 izz="1.0e-06" />
+                iyy="1.0e-06" iyz="0.0"
+                izz="1.0e-06" />
       </inertial>
     </link>
     <joint name="${prefix}end_effector_joint" type="fixed">
-      <parent link="${prefix}link5"/>
+      <parent link="${prefix}link7"/>
       <child link="${prefix}end_effector_link"/>
-      <origin xyz="0.126 0.0 0.0" rpy="0 0 0"/>
+      <origin xyz="0.0 0.0 0.115" rpy="0 0 0"/>
     </joint>
     <link name="${prefix}end_effector_link">
@@ -225,5 +283,5 @@
         </geometry>
         <material name="red"/>
-       </visual>
+      </visual>
     </link>
   </xacro:macro>

File: open_manipulator_x_moveit_config/config/open_manipulator_x.ros2_control.xacro (robot description, xacro)
@@ -36,4 +36,18 @@
                 <state_interface name="velocity"/>
             </joint>
+            <joint name="joint5">
+                <command_interface name="position"/>
+                <state_interface name="position">
+                  <param name="initial_value">${initial_positions['joint5']}</param>
+                </state_interface>
+                <state_interface name="velocity"/>
+            </joint>
+            <joint name="joint6">
+                <command_interface name="position"/>
+                <state_interface name="position">
+                  <param name="initial_value">${initial_positions['joint6']}</param>
+                </state_interface>
+                <state_interface name="velocity"/>
+            </joint>
             <joint name="gripper_left_joint">
                 <command_interface name="position"/>
